File: board/SSR10A.kicad_pcb (KiCad board)
At the start: 2 copper layers, 182 x 48 mm, 100 parts, among them J1 1, J10 9, J2 0, J3 2, J4 3, J5 4, J6 5, J7 6, J8 7, J9 8, U1 HLK-PM03, U10 MOC306XMS, U11 MOC306XMS, U12 MOC306XMS, U13 MOC306XMS, U2 PY32F030K1xTx, U3 PAN2110P0AA, U4 MOC306XMS, U5 MOC306XMS, U6 MOC306XMS, U7 MOC306XMS, U8 MOC306XMS, U9 MOC306XMS, X1 SWD, Y1 16MHz

Commit message: Refactor code structure for improved readability and maintainability
Parts:
- removed D10, D11, D4, D5, D6, D7, D8, D9: BTA08S-600CW, Package_TO_SOT_SMD:TO-252-2
- removed the D3 at (145.5, 63.4)
- removed J10: 9, Drake:DG235-3.81-02P
- removed J2: 0, Drake:DG235-3.81-02P
- removed J3: 2, Drake:DG235-3.81-02P
- removed J4: 3, Drake:DG235-3.81-02P
- removed J5: 4, Drake:DG235-3.81-02P
- removed J6: 5, Drake:DG235-3.81-02P
- removed J7: 6, Drake:DG235-3.81-02P
- removed J8: 7, Drake:DG235-3.81-02P
- removed J9: 8, Drake:DG235-3.81-02P
- removed R10, R11, R12, R15, R16, R17, R20, R21, R22, R25, R26, R27, R30, R31, R32, R35, R36, R37, R40, R41, R42, R45, R46, R47, R50, R51, R52: 680R, Resistor_SMD:R_0805_2012Metric
- removed R13, R18, R23, R28, R33, R38, R43, R48, R8: 10k, Resistor_SMD:R_0805_2012Metric
- removed R14, R19, R24, R29, R34, R39, R44, R49, R9: 270R, Resistor_SMD:R_0805_2012Metric
- removed U10, U11, U12, U13, U5, U6, U7, U8, U9: MOC306XMS, Package_DIP:SMDIP-4_W7.62mm
- added D2: LED, LED_SMD:LED_0805_2012Metric_Pad1.15x1.40mm_HandSolder, F.Cu at (79.0, 99.0)
- IN1: value Conn_01x02 -> MAINS; footprint Drake:DG235-3.81-02P -> Connector_Phoenix_MSTB:PhoenixContact_MSTBA_2,5_3-G_1x03_P5.00mm_Horizontal
- J1: value 1 -> 0; footprint Drake:DG235-3.81-02P -> Connector_Phoenix_MSTB:PhoenixContact_MSTBA_2,5_3-G_1x03_P5.00mm_Horizontal
- R1: value 270R -> 330R
- R3: value 10k -> 330R
- RV1: moved to B.Cu
- moved U4 169.5 mm to (74.0, 103.0), turned to -90 degrees
- moved R7 165.3 mm to (72.0, 112.5), turned to 180 degrees
- moved J1 164.2 mm to (72.0, 121.2)
- moved R6 163.0 mm to (72.0, 110.5)
- moved D3 159.8 mm to (79.7, 112.4), turned to 180 degrees
- moved R4 157.5 mm to (74.0, 96.0), turned to 180 degrees
- moved R3 154.2 mm to (79.0, 96.0)
- moved R5 151.0 mm to (85.0, 112.5), turned to -90 degrees
- moved D1 108.5 mm to (74.0, 77.0)
- moved R1 108.5 mm to (78.5, 77.0)
- moved H1 108.2 mm to (24.0, 28.0)
- moved C6 86.9 mm to (57.0, 64.0)
- moved U1 59.4 mm to (125.0, 57.0)
- moved H2 52.7 mm to (20.0, 43.0)
- moved IN1 6.44 mm to (54.0, 121.2)
- renumbered D2 to D3, R7 to R5, R5 to R7
Connections:
- D3 pad 1: MAINS-N -> MAINS-L
- D3 pad 3: Net-(D2-G) -> Net-(D3-G)
- IN1 pad 1: MAINS-N -> MAINS-L
- IN1 pad 2: MAINS-L -> MAINS-N
- J1 pad 2: MAINS-L -> MAINS-N
- R3 pad 1: ~{CH1} -> ~{CH0}
- R3 pad 2: +3V3 -> Net-(D2-K)
- R4 pad 1: ~{CH1} -> ~{CH0}
- R5 pad 1: Net-(D2-G) -> Net-(D3-G)
- R5 pad 2: MAINS-N -> MAINS-L
- R6 pad 1: Net-(R5-Pad2) -> Net-(R6-Pad1)
- R7 pad 2: Net-(R5-Pad2) -> Net-(R6-Pad1)
- RV1 pad 1: MAINS-L -> MAINS-N
- RV1 pad 2: MAINS-N -> MAINS-L
- U1 pad 1: MAINS-L -> MAINS-N
- U1 pad 2: MAINS-N -> MAINS-L
- U4 pad 3: Net-(D2-G) -> Net-(R6-Pad1)
- U4 pad 4: Net-(R5-Pad2) -> Net-(D3-G)
Routing:
- net (no net): track 1560.3 -> 0.00 mm, vias 10 -> 0
- net +3V3: track 363.6 -> 4.32 mm, vias 1 -> 0
- net /LED: track 31.7 -> 0.00 mm, vias 2 -> 0
- net Net-(D3-A2) (its old number): track 19.3 -> 0.00 mm
- net Net-(D3-A2): track 0.00 -> 15.1 mm, vias 0 -> 8
- net Net-(D3-G): track 0.00 -> 11.8 mm
- net ~{CH0}: track 0.00 -> 8.35 mm
- net Net-(R6-Pad1): track 0.00 -> 6.37 mm
- net MAINS-PE: track 0.00 -> 4.78 mm
- net MAINS-N: track 0.00 -> 4.78 mm
- net GND: track 3.83 -> 0.00 mm, vias 78 -> 0
- net Net-(R4-Pad2): track 0.00 -> 3.34 mm
- net Net-(D2-K): track 0.00 -> 3.05 mm
- net MAINS-L: track 0.00 -> 2.49 mm, vias 0 -> 2
- net Net-(D1-A): track 2.47 -> 0.00 mm
- added copper zone on B.Cu, net Net-(D3-A2)
- added copper zone on F.Cu, net Net-(D3-A2)
- removed copper zone on B.Cu, net GND
- removed copper zone on F.Cu, net GND
Other:
- board size 182 x 48 mm -> 214 x 48 mm
- board text added: "bleriot-SSR10A v1.0 drake.cz"
- board text removed: "1"
- board text removed: "2"
- board text removed: "3"
- board text removed: "4"
- board text removed: "5"
- board text removed: "6"
- board text removed: "7"
- board text removed: "SSR10A v3.0 Bleriot drake.cz Max load: 2A/channel"

Commit message: Refactor code structure for improved readability and maintainability
Parts:
- removed A1: 31mm, RF_Antenna:Texas_SWRA117D_2.4GHz_Right
- removed C1, C4: 1u, Capacitor_SMD:C_0805_2012Metric
- removed C2, C3, C5, C7: 100n, Capacitor_SMD:C_0805_2012Metric
- removed C6: 47u, Capacitor_SMD:C_0805_2012Metric
- removed D1, D2: LED, LED_SMD:LED_0805_2012Metric_Pad1.15x1.40mm_HandSolder
- removed D3: BTA08S-600CW, Package_TO_SOT_SMD:TO-252-2
- removed H1, H2: MountingHole, MountingHole:MountingHole_3.7mm_Pad_Via
- removed J1: 0, Connector_Phoenix_MSTB:PhoenixContact_MSTBA_2,5_3-G_1x03_P5.00mm_Horizontal
- removed R1, R3: 330R, Resistor_SMD:R_0805_2012Metric
- removed R2: 10k, Resistor_SMD:R_0805_2012Metric
- removed R4: 270R, Resistor_SMD:R_0805_2012Metric
- removed R5, R6, R7: 680R, Resistor_SMD:R_0805_2012Metric
- removed U1: HLK-PM03, Drake:HLK-PM01
- removed U2: PY32F030K1xTx, Package_QFP:LQFP-32_7x7mm_P0.8mm
- removed U3: PAN2110P0AA, Package_SO:SOIC-8_3.9x4.9mm_P1.27mm
- removed U4: MOC306XMS, Package_DIP:SMDIP-4_W7.62mm
- removed X1: SWD, Drake:SWD
- removed Y1: 16MHz, Crystal:Crystal_SMD_3225-4Pin_3.2x2.5mm
Routing:
- net Net-(D3-A2): track 15.1 -> 0.00 mm, vias 8 -> 0
- net Net-(D3-G): track 11.8 -> 0.00 mm
- net ~{CH0}: track 8.35 -> 0.00 mm
- net Net-(R6-Pad1): track 6.37 -> 0.00 mm
- net MAINS-PE: track 4.78 -> 0.00 mm
- net MAINS-N: track 4.78 -> 0.00 mm
- net +3V3: track 4.32 -> 0.00 mm
- net Net-(R4-Pad2): track 3.34 -> 0.00 mm
- net Net-(D2-K): track 3.05 -> 0.00 mm
- net MAINS-L: track 2.49 -> 0.00 mm, vias 2 -> 0
- removed copper zone on B.Cu, net Net-(D3-A2)
- removed copper zone on F.Cu, net Net-(D3-A2)
Other:
- outline, holes or cut-outs redrawn
- board text removed: "CHANNEL"

Commit message: WIP
Parts:
- added A1: 31mm, RF_Antenna:Texas_SWRA117D_2.4GHz_Right, F.Cu at (214.4, 122.5)
- added C1: 1u, Capacitor_SMD:C_0805_2012Metric, F.Cu at (203.3, 123.5)
- added C2: 100n, Capacitor_SMD:C_0805_2012Metric, F.Cu at (200.3, 123.5)
- added C3: 1u, Capacitor_SMD:C_0805_2012Metric, F.Cu at (196.1, 94.0)
- added C4: 100n, Capacitor_SMD:C_0805_2012Metric, F.Cu at (196.1, 97.0)
- added C5: 100n, Capacitor_SMD:C_0805_2012Metric, F.Cu at (195.5, 111.0)
- added C6: 47u, Capacitor_SMD:C_0805_2012Metric, F.Cu at (174.0, 98.5)
- added C7: 100n, Capacitor_SMD:C_0805_2012Metric, F.Cu at (182.5, 107.0)
- added D1: LED, LED_SMD:LED_0805_2012Metric_Pad1.15x1.40mm_HandSolder, F.Cu at (201.0, 99.0)
- added D10: LED, LED_SMD:LED_0805_2012Metric_Pad1.15x1.40mm_HandSolder, F.Cu at (151.0, 99.0)
- added D11: BTA08S-600CW, Package_TO_SOT_SMD:TO-252-2, F.Cu at (151.7, 112.4)
- added D2: LED, LED_SMD:LED_0805_2012Metric_Pad1.15x1.40mm_HandSolder, F.Cu at (79.0, 99.0)
- added D3: BTA08S-600CW, Package_TO_SOT_SMD:TO-252-2, F.Cu at (79.7, 112.4)
- added D4: LED, LED_SMD:LED_0805_2012Metric_Pad1.15x1.40mm_HandSolder, F.Cu at (97.0, 99.0)
- added D5: BTA08S-600CW, Package_TO_SOT_SMD:TO-252-2, F.Cu at (97.7, 112.4)
- added D6: LED, LED_SMD:LED_0805_2012Metric_Pad1.15x1.40mm_HandSolder, F.Cu at (115.0, 99.0)
- added D7: BTA08S-600CW, Package_TO_SOT_SMD:TO-252-2, F.Cu at (115.7, 112.4)
- added D8: LED, LED_SMD:LED_0805_2012Metric_Pad1.15x1.40mm_HandSolder, F.Cu at (133.0, 99.0)
- added D9: BTA08S-600CW, Package_TO_SOT_SMD:TO-252-2, F.Cu at (133.7, 112.4)
- added H1: MountingHole, MountingHole:MountingHole_3.7mm_Pad_Via, F.Cu at (56.0, 110.0)
- added H2: MountingHole, MountingHole:MountingHole_3.7mm_Pad_Via, F.Cu at (214.0, 110.0)
- added J1: 0, Connector_Phoenix_MSTB:PhoenixContact_MSTBA_2,5_3-G_1x03_P5.00mm_Horizontal, F.Cu at (72.0, 121.2)
- added J2: 1, Connector_Phoenix_MSTB:PhoenixContact_MSTBA_2,5_3-G_1x03_P5.00mm_Horizontal, F.Cu at (90.0, 121.2)
- added J3: 2, Connector_Phoenix_MSTB:PhoenixContact_MSTBA_2,5_3-G_1x03_P5.00mm_Horizontal, F.Cu at (108.0, 121.2)
- added J4: 3, Connector_Phoenix_MSTB:PhoenixContact_MSTBA_2,5_3-G_1x03_P5.00mm_Horizontal, F.Cu at (126.0, 121.2)
- added J5: 4, Connector_Phoenix_MSTB:PhoenixContact_MSTBA_2,5_3-G_1x03_P5.00mm_Horizontal, F.Cu at (144.0, 121.2)
- added R1: 10k, Resistor_SMD:R_0805_2012Metric, F.Cu at (209.9, 131.4)
- added R10: 680R, Resistor_SMD:R_0805_2012Metric, F.Cu at (103.0, 112.5)
- added R11: 680R, Resistor_SMD:R_0805_2012Metric, F.Cu at (90.0, 110.5)
- added R12: 680R, Resistor_SMD:R_0805_2012Metric, F.Cu at (90.0, 112.5)
- added R13: 330R, Resistor_SMD:R_0805_2012Metric, F.Cu at (115.0, 96.0)
- added R14: 270R, Resistor_SMD:R_0805_2012Metric, F.Cu at (110.0, 96.0)
- added R15: 680R, Resistor_SMD:R_0805_2012Metric, F.Cu at (121.0, 112.5)
- added R16: 680R, Resistor_SMD:R_0805_2012Metric, F.Cu at (108.0, 110.5)
- added R17: 680R, Resistor_SMD:R_0805_2012Metric, F.Cu at (108.0, 112.5)
- added R18: 330R, Resistor_SMD:R_0805_2012Metric, F.Cu at (133.0, 96.0)
- added R19: 270R, Resistor_SMD:R_0805_2012Metric, F.Cu at (128.0, 96.0)
- added R2: 330R, Resistor_SMD:R_0805_2012Metric, F.Cu at (201.0, 102.0)
- added R20: 680R, Resistor_SMD:R_0805_2012Metric, F.Cu at (139.0, 112.5)
- added R21: 680R, Resistor_SMD:R_0805_2012Metric, F.Cu at (126.0, 110.5)
- added R22: 680R, Resistor_SMD:R_0805_2012Metric, F.Cu at (126.0, 112.5)
- added R23: 330R, Resistor_SMD:R_0805_2012Metric, F.Cu at (151.0, 96.0)
- added R24: 270R, Resistor_SMD:R_0805_2012Metric, F.Cu at (146.0, 96.0)
- added R25: 680R, Resistor_SMD:R_0805_2012Metric, F.Cu at (157.0, 112.5)
- added R26: 680R, Resistor_SMD:R_0805_2012Metric, F.Cu at (144.0, 110.5)
- added R27: 680R, Resistor_SMD:R_0805_2012Metric, F.Cu at (144.0, 112.5)
- added R3: 330R, Resistor_SMD:R_0805_2012Metric, F.Cu at (79.0, 96.0)
- added R4: 270R, Resistor_SMD:R_0805_2012Metric, F.Cu at (74.0, 96.0)
- added R5: 680R, Resistor_SMD:R_0805_2012Metric, F.Cu at (85.0, 112.5)
- added R6: 680R, Resistor_SMD:R_0805_2012Metric, F.Cu at (72.0, 110.5)
- added R7: 680R, Resistor_SMD:R_0805_2012Metric, F.Cu at (72.0, 112.5)
- added R8: 330R, Resistor_SMD:R_0805_2012Metric, F.Cu at (97.0, 96.0)
- added R9: 270R, Resistor_SMD:R_0805_2012Metric, F.Cu at (92.0, 96.0)
- added U1: PAN2110P0AA, Package_SO:SOIC-8_3.9x4.9mm_P1.27mm, F.Cu at (208.0, 120.0)
- added U2: HLK-PM03, Drake:HLK-PM01, F.Cu at (170.0, 118.0)
- added U3: PY32F030K1xTx, Package_QFP:LQFP-32_7x7mm_P0.8mm, F.Cu at (190.0, 103.0)
- added U4: MOC306XMS, Package_DIP:SMDIP-4_W7.62mm, F.Cu at (74.0, 103.0)
- added U5: MOC306XMS, Package_DIP:SMDIP-4_W7.62mm, F.Cu at (92.0, 103.0)
- added U6: MOC306XMS, Package_DIP:SMDIP-4_W7.62mm, F.Cu at (110.0, 103.0)
- added U7: MOC306XMS, Package_DIP:SMDIP-4_W7.62mm, F.Cu at (128.0, 103.0)
- added U8: MOC306XMS, Package_DIP:SMDIP-4_W7.62mm, F.Cu at (146.0, 103.0)
- added X1: SWD, Drake:SWD, F.Cu at (190.0, 91.0)
- added Y1: 16MHz, Crystal:Crystal_SMD_3225-4Pin_3.2x2.5mm, F.Cu at (203.2, 131.8)
- moved RV1 17.0 mm to (56.6, 126.0), turned to 180 degrees
Routing:
- net MAINS-L: track 0.00 -> 151.7 mm, vias 0 -> 10
- net MAINS-N: track 0.00 -> 141.8 mm
- net +3V3: track 0.00 -> 124.6 mm
- net MAINS-PE: track 0.00 -> 118.1 mm
- net ~{CH0}: track 0.00 -> 110.8 mm
- net ~{CH1}: track 0.00 -> 91.0 mm
- net ~{CH2}: track 0.00 -> 71.9 mm
- net ~{CH3}: track 0.00 -> 53.3 mm
- net ~{CH4}: track 0.00 -> 35.4 mm
- net Net-(D11-A2): track 0.00 -> 15.1 mm, vias 0 -> 8
- net Net-(D9-A2): track 0.00 -> 12.5 mm, vias 0 -> 8
- net Net-(D7-A2): track 0.00 -> 12.5 mm, vias 0 -> 8
- net Net-(D5-A2): track 0.00 -> 12.5 mm, vias 0 -> 8
- net Net-(D3-A2): track 0.00 -> 12.5 mm, vias 0 -> 8
- net Net-(D9-G): track 0.00 -> 11.8 mm
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- added copper zone on B.Cu, net Net-(D11-A2)
- added copper zone on F.Cu, net Net-(D11-A2)
- added copper zone on F.Cu, net Net-(D3-A2)
- added copper zone on F.Cu, net Net-(D5-A2)
- added copper zone on F.Cu, net Net-(D7-A2)
- added copper zone on F.Cu, net Net-(D9-A2)
Other:
- board size 214 x 48 mm -> 170 x 48 mm
- board text added: "CHANNEL"

Commit message: WIP
Parts:
- J1: value 0 -> 1
- J2: value 1 -> 2
- J3: value 2 -> 3
- J4: value 3 -> 4
- J5: value 4 -> 5
- moved U2 74.2 mm to (98.0, 100.0), turned to 0 degrees
- moved C6 57.3 mm to (117.0, 93.0), turned to 90 degrees
- moved D10 47.5 mm to (198.5, 99.0)
- moved D11 47.5 mm to (199.2, 112.4)
- moved D2 47.5 mm to (126.5, 99.0)
- moved D3 47.5 mm to (127.2, 112.4)
- moved D4 47.5 mm to (144.5, 99.0)
- moved D5 47.5 mm to (145.2, 112.4)
- moved D6 47.5 mm to (162.5, 99.0)
- moved D7 47.5 mm to (163.2, 112.4)
- moved D8 47.5 mm to (180.5, 99.0)
- moved D9 47.5 mm to (181.2, 112.4)
- moved IN1 47.5 mm to (101.5, 121.2)
- moved J1 47.5 mm to (119.5, 121.2)
- moved J2 47.5 mm to (137.5, 121.2)
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Connections:
- R13 pad 1: ~{CH2} -> ~{CH3}
- R14 pad 1: ~{CH2} -> ~{CH3}
- R18 pad 1: ~{CH3} -> ~{CH4}
- R19 pad 1: ~{CH3} -> ~{CH4}
- R23 pad 1: ~{CH4} -> ~{CH5}
- R24 pad 1: ~{CH4} -> ~{CH5}
- R3 pad 1: ~{CH0} -> ~{CH1}
- R4 pad 1: ~{CH0} -> ~{CH1}
- R8 pad 1: ~{CH1} -> ~{CH2}
- R9 pad 1: ~{CH1} -> ~{CH2}
- U3 pad 19: ~{CH0} -> unconnected-(U3-PA9-OSC32OUT-Pad19)
- U3 pad 20: ~{CH1} -> unconnected-(U3-PA10-OSC32IN-Pad20)
- U3 pad 21: ~{CH2} -> ~{CH1}
- U3 pad 22: ~{CH3} -> ~{CH2}
- U3 pad 25: ~{CH4} -> ~{CH3}
- U3 pad 26: ~{CH5} -> ~{CH4}
- U3 pad 27: ~{CH6} -> ~{CH5}
- U3 pad 28: ~{CH7} -> unconnected-(U3-PB5-Pad28)
- U3 pad 29: ~{CH8} -> unconnected-(U3-PB6-Pad29)
- U3 pad 30: ~{CH9} -> unconnected-(U3-PB7-Pad30)
Routing:
- net ~{CH0}: track 110.8 -> 0.00 mm
- net +3V3: track 124.6 -> 198.2 mm
- net ~{CH5}: track 0.00 -> 23.7 mm
- net /~{RF_CS}: track 0.00 -> 21.3 mm, vias 0 -> 2
- net /RF_DATA: track 0.00 -> 20.5 mm, vias 0 -> 3
- net Net-(U3-PA14-SWC): track 0.00 -> 19.2 mm, vias 0 -> 2
- net MAINS-N: track 141.8 -> 159.4 mm
- net /RF_SCK: track 0.00 -> 17.5 mm, vias 0 -> 2
- net Net-(U3-PA13-SWD): track 0.00 -> 14.7 mm, vias 0 -> 2
- net ~{CH1}: track 91.0 -> 102.3 mm
- net ~{CH2}: track 71.9 -> 82.5 mm
- net /LED: track 0.00 -> 10.7 mm, vias 0 -> 2
- net ~{CH3}: track 53.3 -> 60.7 mm
- net ~{CH4}: track 35.4 -> 42.2 mm
- net Net-(U1-XC0): track 0.00 -> 5.80 mm
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Other:
- board size 170 x 48 mm -> 150 x 48 mm
