File: board/SSR10A.kicad_sch (KiCad schematic)
At the start: 20 parts, among them U1 HLK-PM03, U2 PY32F030K1xTx, U3 PAN2110P0AA, X1 SWD, Y1 16MHz

Commit message: Refactor code structure for improved readability and maintainability
Parts:
- removed IN1: Conn_01x02, Drake:DG235-3.81-02P, symbol Connector_Generic:Conn_01x02
- added IN1: MAINS, Connector_Phoenix_MSTB:PhoenixContact_MSTBA_2,5_3-G_1x03_P5.00mm_Horizontal, symbol Connector_Generic:Conn_01x03
- R2: renamed from R1; value 270R -> 330R
- renumbered C4 to C1, C5 to C2, C1 to C3, C2 to C4, C3 to C5, R2 to R1, U3 to U1, U1 to U2, U2 to U3
Connections:
- net MAINS-L: now also RV1.2, U2.2 (LINE2), IN1.1 (Pin_1); no longer RV1.1, U2.1 (LINE1)
- net MAINS-N: now also RV1.1, U2.1 (LINE1), IN1.2 (Pin_2); no longer RV1.2, U2.2 (LINE2)
- new net MAINS-PE: IN1.3 (Pin_3)
Other:
- removed sheet ssr-channel-${Channel}
- moved on the sheet: A1, C1, C2, C3, C4, C5, C6, C7, D1, H1, H2, R1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

Commit message: Refactor code structure for improved readability and maintainability
Other:
- added sheet ssr-channel0 (ssr-channel.kicad_sch)
- added sheet ssr-channel1 (ssr-channel.kicad_sch)
Changed lines of the file:
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@@
+		)
+	)
+	(sheet
+		(at 52.07 180.34)
+		(size 12.7 3.81)
+		(exclude_from_sim no)
+		(in_bom yes)
+		(on_board yes)
+		(dnp no)
+		(fields_autoplaced yes)
+		(stroke
+			(width 0.1524)
+			(type solid)
+		)
+		(fill
+			(color 0 0 0 0)
+		)
+		(property "Sheetname" "ssr-channel1"
+			(at 52.07 179.5014 0)
+			(show_name no)
+			(do_not_autoplace no)
+			(effects
+				(font
+					(size 1.524 1.524)
+				)
+				(justify left bottom)
+			)
+		)
+		(property "Sheetfile" "ssr-channel.kicad_sch"
+			(at 52.07 184.8362 0)
+			(show_name no)
+			(do_not_autoplace no)
+			(effects
+				(font
+					(size 1.524 1.524)
+				)
+				(justify left top)
+			)
+		)
+		(property "Channel" "1"
+			(at 0 10.16 0)
+			(hide yes)
+			(show_name no)
+			(do_not_autoplace no)
+			(effects
+				(font
+					(size 1.524 1.524)
+				)
+			)
+		)
+		(instances
+			(project "SSR10A"
+				(path "/6b7dd4b9-634f-41b4-b846-9b2e2d6d43c6"
+					(page "3")
+				)
+			)
+		)
+	)
+	(sheet
+		(at 52.07 170.18)
+		(size 12.7 3.81)
+		(exclude_from_sim no)
+		(in_bom yes)
+		(on_board yes)
+		(dnp no)
+		(fields_autoplaced yes)
+		(stroke
+			(width 0.1524)
+			(type solid)
+		)
+		(fill
+			(color 0 0 0 0)
+		)
+		(property "Sheetname" "ssr-channel0"
+			(at 52.07 169.3414 0)
+			(show_name no)
+			(do_not_autoplace no)
+			(effects
+				(font
+					(size 1.524 1.524)
+				)
+				(justify left bottom)
+			)
+		)
+		(property "Sheetfile" "ssr-channel.kicad_sch"
+			(at 52.07 174.6762 0)
+			(show_name no)
+			(do_not_autoplace no)
+			(effects
+				(font
+					(size 1.524 1.524)
+				)
+				(justify left top)
+			)
+		)
+		(property "Channel" "0"
+			(at 0 0 0)
+			(hide yes)
+			(show_name no)
+			(do_not_autoplace no)
+			(effects
+				(font
+					(size 1.524 1.524)
+				)
+			)
+		)
+		(instances
+			(project "SSR10A"
+				(path "/6b7dd4b9-634f-41b4-b846-9b2e2d6d43c6"
+					(page "2")
+				)
+			)
 		)
 	)

Commit message: WIP
Other:
- added sheet ssr-channel2 (ssr-channel.kicad_sch)
- added sheet ssr-channel3 (ssr-channel.kicad_sch)
- added sheet ssr-channel4 (ssr-channel.kicad_sch)
- moved on the sheet: D1, H1, H2, R2

Commit message: WIP
Connections:
- net ~{CH6} is gone; now on net ~{CH5}: U3.27 (PB4)
- net ~{CH1}: now also U3.21 (PA11); no longer U3.20 (PA10-OSC32IN)
- net ~{CH2}: now also U3.22 (PA12); no longer U3.21 (PA11)
- net ~{CH3}: now also U3.25 (PA15); no longer U3.22 (PA12)
- net ~{CH4}: now also U3.26 (PB3); no longer U3.25 (PA15)
- net ~{CH5}: no longer U3.26 (PB3)
- net ~{CH0}: no longer names the net of U3.19 (PA9-OSC32OUT)
- net ~{CH7}: no longer names the net of U3.28 (PB5)
- net ~{CH8}: no longer names the net of U3.29 (PB6)
- net ~{CH9}: no longer names the net of U3.30 (PB7)
- no-connect marks 11 -> 16
Other:
- sheet ssr-channel0 renamed channel1
- sheet ssr-channel1 renamed channel2
- sheet ssr-channel2 renamed channel3
- sheet ssr-channel3 renamed channel4
- sheet ssr-channel4 renamed channel5
Changed lines of the file:
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@@
 	)
 	(no_connect
+		(at 200.66 76.2)
+	)
+	(no_connect
 		(at 198.12 76.2)
 	)
@@
 	)
 	(no_connect
+		(at 226.06 101.6)
+	)
+	(no_connect
 		(at 182.88 106.68)
 	)
+	(no_connect
+		(at 226.06 99.06)
+	)
+	(no_connect
+		(at 203.2 76.2)
+	)
+	(no_connect
+		(at 205.74 76.2)
+	)
 	(wire
 		(pts
@@
 		)
 	)
-	(global_label "~{CH7}"
-		(shape input)
-		(at 205.74 76.2 90)
-		(fields_autoplaced yes)
-		(effects
-			(font
-				(size 1.524 1.524)
-			)
-			(justify left)
-		)
-		(property "Intersheetrefs" "${INTERSHEET_REFS}"
-			(at 205.74 68.8312 90)
-			(hide yes)
-			(show_name no)
-			(do_not_autoplace no)
-			(effects
-				(font
-					(size 1.27 1.27)
-				)
-				(justify left)
-			)
-		)
-	)
 	(global_label "MAINS-L"
 		(shape input)
@@
 	(global_label "~{CH5}"
 		(shape input)
-		(at 210.82 76.2 90)
-		(fields_autoplaced yes)
-		(effects
-			(font
-				(size 1.524 1.524)
-			)
-			(justify left)
-		)
-		(property "Intersheetrefs" "${INTERSHEET_REFS}"
-			(at 210.82 68.8312 90)
-			(hide yes)
-			(show_name no)
-			(do_not_autoplace no)
-			(effects
-				(font
-					(size 1.27 1.27)
-				)
-				(justify left)
-			)
-		)
-	)
-	(global_label "~{CH8}"
-		(shape input)
-		(at 203.2 76.2 90)
+		(at 208.28 76.2 90)
 		(fields_autoplaced yes)
 		(effects
@@
 		)
 		(property "Intersheetrefs" "${INTERSHEET_REFS}"
-			(at 203.2 68.8312 90)
+			(at 208.28 68.8312 90)
 			(hide yes)
 			(show_name no)
@@
 	(global_label "~{CH3}"
 		(shape input)
-		(at 226.06 93.98 0)
+		(at 213.36 76.2 90)
 		(fields_autoplaced yes)
 		(effects
@@
 		)
 		(property "Intersheetrefs" "${INTERSHEET_REFS}"
-			(at 233.4288 93.98 0)
+			(at 213.36 68.8312 90)
 			(hide yes)
 			(show_name no)
@@
 		)
 	)
-	(global_label "~{CH0}"
-		(shape input)
-		(at 226.06 101.6 0)
-		(fields_autoplaced yes)
-		(effects
-			(font
-				(size 1.524 1.524)
-			)
-			(justify left)
-		)
-		(property "Intersheetrefs" "${INTERSHEET_REFS}"
-			(at 233.4288 101.6 0)
-			(hide yes)
-			(show_name no)
-			(do_not_autoplace no)
-			(effects
-				(font
-					(size 1.27 1.27)
-				)
-				(justify left)
-			)
-		)
-	)
 	(global_label "~{CH2}"
 		(shape input)
-		(at 226.06 96.52 0)
+		(at 226.06 93.98 0)
 		(fields_autoplaced yes)
 		(effects
@@
 		)
 		(property "Intersheetrefs" "${INTERSHEET_REFS}"
-			(at 233.4288 96.52 0)
+			(at 233.4288 93.98 0)
 			(hide yes)
 			(show_name no)
@@
 		)
 	)
-	(global_label "~{CH9}"
-		(shape input)
-		(at 200.66 76.2 90)
-		(fields_autoplaced yes)
-		(effects
-			(font
-				(size 1.524 1.524)
-			)
-			(justify left)
-		)
-		(property "Intersheetrefs" "${INTERSHEET_REFS}"
-			(at 200.66 68.8312 90)
-			(hide yes)
-			(show_name no)
-			(do_not_autoplace no)
-			(effects
-				(font
-					(size 1.27 1.27)
-				)
-				(justify left)
-			)
-		)
-	)
 	(global_label "MAINS-PE"
 		(shape input)
@@
 		)
 	)
-	(global_label "~{CH6}"
-		(shape input)
-		(at 208.28 76.2 90)
-		(fields_autoplaced yes)
-		(effects
-			(font
-				(size 1.524 1.524)
-			)
-			(justify left)
-		)
-		(property "Intersheetrefs" "${INTERSHEET_REFS}"
-			(at 208.28 68.8312 90)
-			(hide yes)
-			(show_name no)
-			(do_not_autoplace no)
-			(effects
-				(font
-					(size 1.27 1.27)
-				)
-				(justify left)
-			)
-		)
-	)
 	(global_label "~{CH4}"
 		(shape input)
-		(at 213.36 76.2 90)
+		(at 210.82 76.2 90)
 		(fields_autoplaced yes)
 		(effects
@@
 		)
 		(property "Intersheetrefs" "${INTERSHEET_REFS}"
-			(at 213.36 68.8312 90)
+			(at 210.82 68.8312 90)
 			(hide yes)
 			(show_name no)
@@
 	(global_label "~{CH1}"
 		(shape input)
-		(at 226.06 99.06 0)
+		(at 226.06 96.52 0)
 		(fields_autoplaced yes)
 		(effects
@@
 		)
 		(property "Intersheetrefs" "${INTERSHEET_REFS}"
-			(at 233.4288 99.06 0)
+			(at 233.4288 96.52 0)
 			(hide yes)
 			(show_name no)
@@
 			(color 0 0 0 0)
 		)
-		(property "Sheetname" "ssr-channel1"
+		(property "Sheetname" "channel2"
 			(at 35.56 151.5614 0)
 			(show_name no)
@@
 			)
 		)
-		(property "Channel" "1"
+		(property "Channel" "2"
 			(at -16.51 -17.78 0)
 			(hide yes)
@@
 			(color 0 0 0 0)
 		)
-		(property "Sheetname" "ssr-channel4"
+		(property "Sheetname" "channel5"
 			(at 35.56 182.0414 0)
 			(show_name no)
@@
 			)
 		)
-		(property "Channel" "4"
+		(property "Channel" "5"
 			(at -16.51 12.7 0)
 			(hide yes)
@@
 			(color 0 0 0 0)
 		)
-		(property "Sheetname" "ssr-channel0"
+		(property "Sheetname" "channel1"
 			(at 35.56 141.4014 0)
 			(show_name no)
@@
 			)
 		)
-		(property "Channel" "0"
+		(property "Channel" "1"
 			(at -16.51 -27.94 0)
 			(hide yes)
@@
 			(color 0 0 0 0)
 		)
-		(property "Sheetname" "ssr-channel3"
+		(property "Sheetname" "channel4"
 			(at 35.56 171.8814 0)
 			(show_name no)
@@
 			)
 		)
-		(property "Channel" "3"
+		(property "Channel" "4"
 			(at -16.51 2.54 0)
 			(hide yes)
@@
 			(color 0 0 0 0)
 		)
-		(property "Sheetname" "ssr-channel2"
+		(property "Sheetname" "channel3"
 			(at 35.56 161.7214 0)
 			(show_name no)
@@
 			)
 		)
-		(property "Channel" "2"
+		(property "Channel" "3"
 			(at -16.51 -7.62 0)
 			(hide yes)
