File: board/SSR5A.kicad_pcb (KiCad board)
At the start: 2 copper layers, 150 x 48 mm, 65 parts, among them J1 1, J2 2, J3 3, J4 4, J5 5, U1 PAN2110P0AA, U2 HLK-PM03, U3 PY32F030K1xTx, U4 MOC306XMS, U5 MOC306XMS, U6 MOC306XMS, U7 MOC306XMS, U8 MOC306XMS, X1 SWD, Y1 16MHz

Commit message: WIP
Parts:
- A1: value 31mm -> Antenna_Shield
- moved C1 1.85 mm to (217.9, 121.0)
- moved C2 1.85 mm to (217.9, 119.0)
- moved U1 1.85 mm to (223.9, 124.0)
- moved Y1 1.85 mm to (217.9, 125.0)
Connections:
- A1 pad 2: (no net) -> GND
Routing:
- net GND: track 0.00 -> 23.2 mm, vias 0 -> 75
- net /~{RF_CS}: track 21.3 -> 19.5 mm
- net Net-(A1-A): track 2.58 -> 4.41 mm
- net /RF_SCK: track 17.5 -> 15.6 mm
- net /RF_DATA: track 20.5 -> 18.7 mm
- net +3V3: track 198.2 -> 196.4 mm
- added copper zone on B.Cu, net GND
- added copper zone on F.Cu, net GND
Other:
- board text added: "bleriot-SSR5A v1.0 drake.cz"
- board text removed: "bleriot-SSR10A v1.0 drake.cz"
