File: board/SSR5A.kicad_pcb (KiCad board)
At the start: 2 copper layers, 150 x 48 mm, 65 parts, among them J1 1, J2 2, J3 3, J4 4, J5 5, U1 PAN2110P0AA, U2 HLK-PM03, U3 PY32F030K1xTx, U4 MOC306XMS, U5 MOC306XMS, U6 MOC306XMS, U7 MOC306XMS, U8 MOC306XMS, X1 SWD, Y1 16MHz

Commit message: Add RGB status LED to SSR5A
Co-authored-by: Copilot <223556219+Copilot@users.noreply.github.com>
Copilot-Session: 109a56b3-5fb8-400b-b74c-480b8f593743
Parts:
- removed D1: LED, LED_SMD:LED_0805_2012Metric_Pad1.15x1.40mm_HandSolder
- removed R2: 330R, Resistor_SMD:R_0805_2012Metric
- added D12: WS2812B, LED_SMD:LED_WS2812B_PLCC4_5.0x5.0mm_P3.2mm, F.Cu at (214.0, 95.0)
- added D13: LED, LED_SMD:LED_0805_2012Metric_Pad1.15x1.40mm_HandSolder, F.Cu at (214.0, 95.0)
- added R28: 330R, Resistor_SMD:R_0805_2012Metric, F.Cu at (209.0, 95.0)
Routing:
- net +3V3: track 196.4 -> 208.8 mm
- net /LED: track 10.7 -> 18.8 mm
- net Net-(D13-K): track 0.00 -> 4.35 mm
- net Net-(D1-A): track 4.23 -> 0.00 mm
- net GND: track 23.2 -> 21.7 mm, vias 75 -> 73
- net ~{CH2}: track 82.5 -> 83.2 mm
- net ~{CH1}: track 102.3 -> 102.9 mm
- net /RF_DATA: vias 3 -> 2
- added copper zone on B.Cu, net Net-(D3-A2)
- added copper zone on B.Cu, net Net-(D5-A2)
- added copper zone on B.Cu, net Net-(D7-A2)
- added copper zone on B.Cu, net Net-(D9-A2)
Other:
- board text added: "L - N - PE"
