File: board/SSR5A.kicad_sch (KiCad schematic)
At the start: 20 parts, among them U1 PAN2110P0AA, U2 HLK-PM03, U3 PY32F030K1xTx, X1 SWD, Y1 16MHz

Commit message: WIP
Parts:
- removed A1: 31mm, RF_Antenna:Texas_SWRA117D_2.4GHz_Right, symbol Device:Antenna
- added A1: Antenna_Shield, RF_Antenna:Texas_SWRA117D_2.4GHz_Right, symbol Device:Antenna_Shield
Connections:
- net GND: now also A1.2 (Shield)
- net at U1.8 (ANT): now also A1.1 (A)
